File: main_board/hardware.kicad_sch (KiCad schematic)
At the start: 24 parts, among them J20 Conn_01x02, J21 OLED Pins, M1 OLED

Commit message: After project cleanup
Parts:
- H5, H6: footprint sputterizer:MountingHole_2.5mm-No-Margin -> greenface:MountingHole_2.5mm-No-Margin
- M1: Other (none) -> https://www.amazon.com/gp/product/B072Q2X2LL/; URL https://www.amazon.com/gp/product/B072Q2X2LL/ -> (none)
Changed lines of the file:
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@@
 			)
 		)
-		(property "URL" "https://www.amazon.com/gp/product/B072Q2X2LL/"
+		(property "Other" "https://www.amazon.com/gp/product/B072Q2X2LL/"
 			(at 40.132 156.21 0)
 			(effects
@@
 			)
 		)
-		(property "Footprint" "sputterizer:MountingHole_2.5mm-No-Margin"
+		(property "Footprint" "greenface:MountingHole_2.5mm-No-Margin"
 			(at 19.05 45.085 0)
 			(effects
@@
 			)
 		)
-		(property "Footprint" "sputterizer:MountingHole_2.5mm-No-Margin"
+		(property "Footprint" "greenface:MountingHole_2.5mm-No-Margin"
 			(at 19.05 40.005 0)
 			(effects
