File: main_board/inputs.kicad_sch (KiCad schematic)
At the start: 41 parts, among them J16 3.5mm Jack, J17 3.5mm Jack, U10 TL072CDR, U11 ADS1015IDGS, U12 TL072CDR, U19 TL072CDR

Commit message: After project cleanup
Parts:
- D15, D16, D17, D18, D39, D40, D41, D42: footprint sputterizer:D_SOD-323 -> greenface:D_SOD-323
- J16, J17: footprint audio_jacks:Jack_3.5mm_QingPu_WQP-PJ398SM_Vertical -> greenface:Jack_3.5mm_QingPu_WQP-PJ398SM_Vertical
Changed lines of the file:
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@@
 			)
 		)
-		(property "Footprint" "sputterizer:D_SOD-323"
+		(property "Footprint" "greenface:D_SOD-323"
 			(at 85.725 158.115 0)
 			(effects
@@
 			)
 		)
-		(property "Footprint" "sputterizer:D_SOD-323"
+		(property "Footprint" "greenface:D_SOD-323"
 			(at 84.455 88.9 0)
 			(effects
@@
 			)
 		)
-		(property "Footprint" "sputterizer:D_SOD-323"
+		(property "Footprint" "greenface:D_SOD-323"
 			(at 85.725 147.32 0)
 			(effects
@@
 			)
 		)
-		(property "Footprint" "audio_jacks:Jack_3.5mm_QingPu_WQP-PJ398SM_Vertical"
+		(property "Footprint" "greenface:Jack_3.5mm_QingPu_WQP-PJ398SM_Vertical"
 			(at 66.04 38.1 0)
 			(effects
@@
 			)
 		)
-		(property "Footprint" "sputterizer:D_SOD-323"
+		(property "Footprint" "greenface:D_SOD-323"
 			(at 84.455 78.105 0)
 			(effects
@@
 			)
 		)
-		(property "Footprint" "sputterizer:D_SOD-323"
+		(property "Footprint" "greenface:D_SOD-323"
 			(at 146.05 122.555 0)
 			(effects
@@
 			)
 		)
-		(property "Footprint" "sputterizer:D_SOD-323"
+		(property "Footprint" "greenface:D_SOD-323"
 			(at 146.05 53.34 0)
 			(effects
@@
 			)
 		)
-		(property "Footprint" "sputterizer:D_SOD-323"
+		(property "Footprint" "greenface:D_SOD-323"
 			(at 146.05 41.91 0)
 			(effects
@@
 			)
 		)
-		(property "Footprint" "sputterizer:D_SOD-323"
+		(property "Footprint" "greenface:D_SOD-323"
 			(at 146.05 111.125 0)
 			(effects
@@
 			)
 		)
-		(property "Footprint" "audio_jacks:Jack_3.5mm_QingPu_WQP-PJ398SM_Vertical"
+		(property "Footprint" "greenface:Jack_3.5mm_QingPu_WQP-PJ398SM_Vertical"
 			(at 66.04 107.315 0)
 			(effects
