File: main_board/main_board.kicad_sch (KiCad schematic)
At the start: 75 parts, among them J5 Display Header, J6 EU Power, J7 Conn_01x02_Male, SW10 Push Button, SW11 Push Button, SW12 Push Button, SW13 Push Button, SW14 Push Button, SW15 Push Button, SW16 Push Button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

Commit message: After project cleanup
Parts:
- D13, D14, D19, D45, D46: footprint sputterizer:D_SOD-323 -> greenface:D_SOD-323
- FB1: footprint sputterizer:L_Murata_BLM18P -> greenface:L_Murata_BLM18P
- J5: footprint sputterizer:OLED_Header_Slim -> greenface:OLED_Header_Slim
- SW5: footprint sputterizer:RotaryEncoder_MERP12_24 -> greenface:RotaryEncoder_MERP12_24
- U22: symbol Greenface_Library:LT3502 -> greenface:LT3502
- X1: footprint sputterizer:Oscillator_SMD2520-4P -> greenface:Oscillator_SMD2520-4P
Changed lines of the file:
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@@
 			)
 		)
-		(property "Footprint" "sputterizer:D_SOD-323"
+		(property "Footprint" "greenface:D_SOD-323"
 			(at 214.757 116.967 0)
 			(effects
@@
 			)
 		)
-		(property "Footprint" "sputterizer:D_SOD-323"
+		(property "Footprint" "greenface:D_SOD-323"
 			(at 214.757 122.682 0)
 			(effects
@@
 			)
 		)
-		(property "Footprint" "sputterizer:Oscillator_SMD2520-4P"
+		(property "Footprint" "greenface:Oscillator_SMD2520-4P"
 			(at 45.72 144.78 0)
 			(effects
@@
 	)
 	(symbol
-		(lib_id "Greenface_Library:LT3502")
+		(lib_id "greenface:LT3502")
 		(at 46.228 37.592 0)
 		(unit 1)
@@
 			)
 		)
-		(property "Footprint" "sputterizer:RotaryEncoder_MERP12_24"
+		(property "Footprint" "greenface:RotaryEncoder_MERP12_24"
 			(at 162.052 90.678 0)
 			(effects
@@
 			)
 		)
-		(property "Footprint" "sputterizer:D_SOD-323"
+		(property "Footprint" "greenface:D_SOD-323"
 			(at 214.757 158.242 0)
 			(effects
@@
 			)
 		)
-		(property "Footprint" "sputterizer:OLED_Header_Slim"
+		(property "Footprint" "greenface:OLED_Header_Slim"
 			(at 209.042 93.472 0)
 			(effects
@@
 			)
 		)
-		(property "Footprint" "sputterizer:D_SOD-323"
+		(property "Footprint" "greenface:D_SOD-323"
 			(at 62.738 38.862 90)
 			(effects
@@
 			)
 		)
-		(property "Footprint" "sputterizer:D_SOD-323"
+		(property "Footprint" "greenface:D_SOD-323"
 			(at 214.757 153.797 0)
 			(effects
@@
 			)
 		)
-		(property "Footprint" "sputterizer:L_Murata_BLM18P"
+		(property "Footprint" "greenface:L_Murata_BLM18P"
 			(at 97.536 184.404 90)
 			(effects
