File: main_board/triggers.kicad_sch (KiCad schematic)
At the start: 54 parts, among them J1 3.5mm Jack, J2 3.5mm Jack, J3 3.5mm Jack, J4 3.5mm Jack, Q1 MMBT3904, Q2 MMBT3904, Q3 MMBT3904, Q4 MMBT3904, Q5 MMBT3904, SW1 Push Button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

Commit message: After project cleanup
Parts:
- D1, D2, D3, D4, D5, D6, D7, D8: footprint sputterizer:D_SOD-323 -> greenface:D_SOD-323
- D49: footprint sputterizer:LED_0404 -> greenface:LED_0404
- J1, J2, J3, J4: footprint audio_jacks:Jack_3.5mm_QingPu_WQP-PJ398SM_Vertical -> greenface:Jack_3.5mm_QingPu_WQP-PJ398SM_Vertical
Changed lines of the file:
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@@
 			)
 		)
-		(property "Footprint" "sputterizer:D_SOD-323"
+		(property "Footprint" "greenface:D_SOD-323"
 			(at 149.86 92.71 0)
 			(effects
@@
 			)
 		)
-		(property "Footprint" "sputterizer:D_SOD-323"
+		(property "Footprint" "greenface:D_SOD-323"
 			(at 80.01 45.085 0)
 			(effects
@@
 			)
 		)
-		(property "Footprint" "sputterizer:D_SOD-323"
+		(property "Footprint" "greenface:D_SOD-323"
 			(at 80.01 52.705 0)
 			(effects
@@
 			)
 		)
-		(property "Footprint" "audio_jacks:Jack_3.5mm_QingPu_WQP-PJ398SM_Vertical"
+		(property "Footprint" "greenface:Jack_3.5mm_QingPu_WQP-PJ398SM_Vertical"
 			(at 127 96.52 0)
 			(effects
@@
 			)
 		)
-		(property "Footprint" "sputterizer:D_SOD-323"
+		(property "Footprint" "greenface:D_SOD-323"
 			(at 80.01 101.6 0)
 			(effects
@@
 			)
 		)
-		(property "Footprint" "sputterizer:D_SOD-323"
+		(property "Footprint" "greenface:D_SOD-323"
 			(at 149.86 100.33 0)
 			(effects
@@
 			)
 		)
-		(property "Footprint" "audio_jacks:Jack_3.5mm_QingPu_WQP-PJ398SM_Vertical"
+		(property "Footprint" "greenface:Jack_3.5mm_QingPu_WQP-PJ398SM_Vertical"
 			(at 127 49.53 0)
 			(effects
@@
 			)
 		)
-		(property "Footprint" "sputterizer:LED_0404"
+		(property "Footprint" "greenface:LED_0404"
 			(at 155.194 153.67 0)
 			(effects
@@
 			)
 		)
-		(property "Footprint" "sputterizer:D_SOD-323"
+		(property "Footprint" "greenface:D_SOD-323"
 			(at 149.86 53.34 0)
 			(effects
@@
 			)
 		)
-		(property "Footprint" "sputterizer:D_SOD-323"
+		(property "Footprint" "greenface:D_SOD-323"
 			(at 149.86 45.72 0)
 			(effects
@@
 			)
 		)
-		(property "Footprint" "audio_jacks:Jack_3.5mm_QingPu_WQP-PJ398SM_Vertical"
+		(property "Footprint" "greenface:Jack_3.5mm_QingPu_WQP-PJ398SM_Vertical"
 			(at 57.15 48.895 0)
 			(effects
@@
 			)
 		)
-		(property "Footprint" "sputterizer:D_SOD-323"
+		(property "Footprint" "greenface:D_SOD-323"
 			(at 80.01 93.98 0)
 			(effects
@@
 			)
 		)
-		(property "Footprint" "audio_jacks:Jack_3.5mm_QingPu_WQP-PJ398SM_Vertical"
+		(property "Footprint" "greenface:Jack_3.5mm_QingPu_WQP-PJ398SM_Vertical"
 			(at 57.15 97.79 0)
 			(effects
