File: main_board/usb.kicad_sch (KiCad schematic)
At the start: 6 parts, among them J22 USB-C

Commit message: After project cleanup
Parts:
- J22: footprint sputterizer:CUI_UJ20-C-V-C-3-SMT-TR -> greenface:CUI_UJ20-C-V-C-3-SMT-TR; symbol UJ20-C-V-C-3-SMT-TR:UJ20-C-V-C-3-SMT-TR -> Greenface_Library:USB_20pin; MANUFACTURER (none) -> CUI Devices; MAXIMUM_PACKAGE_HEIGHT (none) -> 10.5mm; PARTREV (none) -> 1.0; STANDARD (none) -> Manufacturer Recommendations
Changed lines of the file:
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@@
 	)
 	(symbol
-		(lib_id "UJ20-C-V-C-3-SMT-TR:UJ20-C-V-C-3-SMT-TR")
+		(lib_id "Greenface_Library:USB_20pin")
 		(at 111.252 74.168 0)
 		(unit 1)
@@
 			)
 		)
-		(property "Footprint" "sputterizer:CUI_UJ20-C-V-C-3-SMT-TR"
+		(property "Footprint" "greenface:CUI_UJ20-C-V-C-3-SMT-TR"
 			(at 111.252 74.168 0)
 			(effects
@@
 				(hide yes)
 			)
+		)
+		(property "PARTREV" "1.0"
+			(at 111.252 74.168 0)
+			(effects
+				(font
+					(size 1.27 1.27)
+				)
+				(justify bottom)
+				(hide yes)
+			)
+		)
+		(property "STANDARD" "Manufacturer Recommendations"
+			(at 111.252 74.168 0)
+			(effects
+				(font
+					(size 1.27 1.27)
+				)
+				(justify bottom)
+				(hide yes)
+			)
+		)
+		(property "MAXIMUM_PACKAGE_HEIGHT" "10.5mm"
+			(at 111.252 74.168 0)
+			(effects
+				(font
+					(size 1.27 1.27)
+				)
+				(justify bottom)
+				(hide yes)
+			)
+		)
+		(property "MANUFACTURER" "CUI Devices"
+			(at 111.252 74.168 0)
+			(effects
+				(font
+					(size 1.27 1.27)
+				)
+				(justify bottom)
+				(hide yes)
+			)
